File: schematic/pcb_left/tangentbord1-left.kicad_pcb (KiCad board)
At the start: 2 copper layers, 129 x 77.5 mm, 26 parts, among them J1 UART, J2 DBG

Commit message: Tweak left PCB, add right & thumb PCB
Parts:
- moved J1 4.28 mm to (147.2, 76.0)
- moved REF** 0.50 mm to (125.5, 77.0)
- moved MCU1 0.41 mm to (140.9, 43.2)
- moved REF** 0.35 mm to (125.5, 33.0)
- moved J2 0.35 mm to (125.5, 58.5)
Connections:
- J1 pad S: /VBUS -> GND
- J1 pad T: GND -> /VBUS
Routing:
- net /VBUS: track 46.4 -> 50.7 mm, vias 1 -> 3
- net Net-(S1-DOUT): track 20.8 -> 24.3 mm
- net /S12: track 116.3 -> 119.2 mm
- net /TX: track 24.5 -> 22.1 mm
- net /S8: track 64.0 -> 61.6 mm
- net /S7: track 86.3 -> 84.0 mm
- net +5V: track 372.0 -> 369.8 mm
- net /RX: track 21.8 -> 19.8 mm
- net /S9: track 41.6 -> 42.5 mm
- net /S5: track 21.1 -> 21.7 mm
- net Net-(J2-Pin_2): track 18.0 -> 18.4 mm, vias 0 -> 1
- net Net-(J2-Pin_3): track 20.3 -> 20.2 mm, vias 0 -> 1
