File: schematic/pcb_left/tk-pie-left.kicad_sch (KiCad schematic)
At the start: 35 parts, among them IC1 PCA9539PW,118, J1 NiceView, J2 Battery Connector, U3 SN74LVC1T45DCK

Commit message: pcb-left: Add through-holes to vbat pads
Connections:
- net GND: no longer C4.2, C5.1, PS1.4 (VSS)
- net VBAT: no longer L2.1
- new net VBAT+: L2.1, U1.VBAT+
- new net VBAT-: C4.2, C5.1, PS1.4 (VSS), U1.VBAT-
- no-connect marks 3 -> 2
Changed lines of the file:
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@@
 	)
 	(junction
-		(at 278.13 262.89)
+		(at 247.65 299.72)
 		(diameter 0)
 		(color 0 0 0 0)
 	)
 	(junction
-		(at 240.03 299.72)
+		(at 278.13 262.89)
 		(diameter 0)
 		(color 0 0 0 0)
 	)
 	(junction
-		(at 252.73 299.72)
+		(at 240.03 299.72)
 		(diameter 0)
 		(color 0 0 0 0)
@@
 		(at 264.16 276.86)
 	)
-	(no_connect
-		(at 273.05 309.88)
-	)
 	(wire
 		(pts
@@
 	(wire
 		(pts
+			(xy 247.65 299.72) (xy 278.13 299.72)
+		)
+		(stroke
+			(width 0)
+			(type default)
+		)
+	)
+	(wire
+		(pts
 			(xy 278.13 262.89) (xy 278.13 281.94)
 		)
@@
 	(wire
 		(pts
-			(xy 240.03 299.72) (xy 252.73 299.72)
-		)
-		(stroke
-			(width 0)
-			(type default)
-		)
-	)
-	(wire
-		(pts
 			(xy 52.07 109.22) (xy 59.69 109.22)
 		)
@@
 	(wire
 		(pts
-			(xy 252.73 299.72) (xy 278.13 299.72)
+			(xy 73.66 144.78) (xy 73.66 162.56)
 		)
 		(stroke
@@
 	(wire
 		(pts
-			(xy 73.66 144.78) (xy 73.66 162.56)
+			(xy 77.47 38.1) (xy 85.09 38.1)
 		)
 		(stroke
@@
 	(wire
 		(pts
-			(xy 77.47 38.1) (xy 85.09 38.1)
+			(xy 283.21 262.89) (xy 278.13 262.89)
 		)
 		(stroke
@@
 	(wire
 		(pts
-			(xy 283.21 262.89) (xy 278.13 262.89)
+			(xy 189.23 73.66) (xy 189.23 109.22)
 		)
 		(stroke
@@
 	(wire
 		(pts
-			(xy 189.23 73.66) (xy 189.23 109.22)
+			(xy 30.48 73.66) (xy 34.29 73.66)
 		)
 		(stroke
@@
 	(wire
 		(pts
-			(xy 30.48 73.66) (xy 34.29 73.66)
+			(xy 240.03 299.72) (xy 247.65 299.72)
 		)
 		(stroke
@@
 		)
 	)
-	(label "VBAT"
-		(at 290.83 262.89 0)
-		(effects
-			(font
-				(size 1.27 1.27)
-			)
-			(justify left bottom)
-		)
-	)
 	(symbol
 		(lib_id "library:MX_SW_SOCKET_RGB")
@@
 	)
 	(symbol
+		(lib_id "power:-BATT")
+		(at 247.65 299.72 180)
+		(unit 1)
+		(exclude_from_sim no)
+		(in_bom yes)
+		(on_board yes)
+		(dnp no)
+		(property "Reference" "#PWR047"
+			(at 247.65 295.91 0)
+			(effects
+				(font
+					(size 1.27 1.27)
+				)
+				(hide yes)
+			)
+		)
+		(property "Value" "VBAT-"
+			(at 247.65 304.292 0)
+			(effects
+				(font
+					(size 1.27 1.27)
+				)
+			)
+		)
+		(property "Footprint" ""
+			(at 247.65 299.72 0)
+			(effects
+				(font
+					(size 1.27 1.27)
+				)
+				(hide yes)
+			)
+		)
+		(property "Datasheet" ""
+			(at 247.65 299.72 0)
+			(effects
+				(font
+					(size 1.27 1.27)
+				)
+				(hide yes)
+			)
+		)
+		(property "Description" "Power symbol creates a global label with name \"-BATT\""
+			(at 247.65 299.72 0)
+			(effects
+				(font
+					(size 1.27 1.27)
+				)
+				(hide yes)
+			)
+		)
+		(pin "1"
+		)
+		(instances
+			(project "tk-pie-left"
+				(path "/9b6bc1bb-4d53-4a7c-b909-4e79c2146edb"
+					(reference "#PWR047")
+					(unit 1)
+				)
+			)
+		)
+	)
+	(symbol
 		(lib_id "power:GND")
 		(at 91.44 116.84 0)
@@
 	)
 	(symbol
+		(lib_id "power:+BATT")
+		(at 290.83 262.89 270)
+		(unit 1)
+		(exclude_from_sim no)
+		(in_bom yes)
+		(on_board yes)
+		(dnp no)
+		(fields_autoplaced yes)
+		(property "Reference" "#PWR066"
+			(at 287.02 262.89 0)
+			(effects
+				(font
+					(size 1.27 1.27)
+				)
+				(hide yes)
+			)
+		)
+		(property "Value" "VBAT+"
+			(at 294.64 262.8899 90)
+			(effects
+				(font
+					(size 1.27 1.27)
+				)
+				(justify left)
+			)
+		)
+		(property "Footprint" ""
+			(at 290.83 262.89 0)
+			(effects
+				(font
+					(size 1.27 1.27)
+				)
+				(hide yes)
+			)
+		)
+		(property "Datasheet" ""
+			(at 290.83 262.89 0)
+			(effects
+				(font
+					(size 1.27 1.27)
+				)
+				(hide yes)
+			)
+		)
+		(property "Description" "Power symbol creates a global label with name \"+BATT\""
+			(at 290.83 262.89 0)
+			(effects
+				(font
+					(size 1.27 1.27)
+				)
+				(hide yes)
+			)
+		)
+		(pin "1"
+		)
+		(instances
+			(project "tk-pie-left"
+				(path "/9b6bc1bb-4d53-4a7c-b909-4e79c2146edb"
+					(reference "#PWR066")
+					(unit 1)
+				)
+			)
+		)
+	)
+	(symbol
 		(lib_id "library:MX_SW_SOCKET_RGB_REV")
 		(at 68.58 69.85 0)
@@
 	)
 	(symbol
-		(lib_id "power:GND")
-		(at 252.73 299.72 0)
+		(lib_id "Connector:Conn_01x01_Pin")
+		(at 68.58 172.72 90)
 		(unit 1)
 		(exclude_from_sim no)
@@
 		(dnp no)
 		(fields_autoplaced yes)
-		(property "Reference" "#PWR075"
-			(at 252.73 306.07 0)
+		(property "Reference" "E1"
+			(at 69.85 172.72 90)
 			(effects
 				(font
 					(size 1.27 1.27)
 				)
-				(hide yes)
+				(justify right)
 			)
 		)
-		(property "Value" "GND"
-			(at 252.73 304.8 0)
+		(property "Value" "Conn_01x01_Pin"
+			(at 67.31 172.085 0)
 			(effects
 				(font
 					(size 1.27 1.27)
 				)
+				(hide yes)
 			)
 		)
-		(property "Footprint" ""
-			(at 252.73 299.72 0)
+		(property "Footprint" "Footprints:Pin0.9mm"
+			(at 68.58 172.72 0)
 			(effects
 				(font
@@
 			)
 		)
-		(property "Datasheet" ""
-			(at 252.73 299.72 0)
+		(property "Datasheet" "~"
+			(at 68.58 172.72 0)
 			(effects
 				(font
@@
 		)
 		(property "Description" ""
-			(at 252.73 299.72 0)
+			(at 68.58 172.72 0)
 			(effects
 				(font
@@
 			(project "tk-pie-left"
 				(path "/9b6bc1bb-4d53-4a7c-b909-4e79c2146edb"
-					(reference "#PWR075")
+					(reference "E1")
 					(unit 1)
 				)
@@
 	)
 	(symbol
-		(lib_id "Connector:Conn_01x01_Pin")
-		(at 68.58 172.72 90)
+		(lib_id "power:-BATT")
+		(at 274.32 27.94 270)
 		(unit 1)
 		(exclude_from_sim no)
@@
 		(on_board yes)
 		(dnp no)
-		(fields_autoplaced yes)
-		(property "Reference" "E1"
-			(at 69.85 172.72 90)
+		(property "Reference" "#PWR071"
+			(at 270.51 27.94 0)
 			(effects
 				(font
 					(size 1.27 1.27)
 				)
-				(justify right)
+				(hide yes)
 			)
 		)
-		(property "Value" "Conn_01x01_Pin"
-			(at 67.31 172.085 0)
+		(property "Value" "VBAT-"
+			(at 281.178 27.94 90)
 			(effects
 				(font
 					(size 1.27 1.27)
 				)
-				(hide yes)
 			)
 		)
-		(property "Footprint" "Footprints:Pin0.9mm"
-			(at 68.58 172.72 0)
+		(property "Footprint" ""
+			(at 274.32 27.94 0)
 			(effects
 				(font
@@
 			)
 		)
-		(property "Datasheet" "~"
-			(at 68.58 172.72 0)
+		(property "Datasheet" ""
+			(at 274.32 27.94 0)
 			(effects
 				(font
@@
 			)
 		)
-		(property "Description" ""
-			(at 68.58 172.72 0)
+		(property "Description" "Power symbol creates a global label with name \"-BATT\""
+			(at 274.32 27.94 0)
 			(effects
 				(font
@@
 		)
 		(instances
-			(project "tk-pie-left"
+			(project ""
 				(path "/9b6bc1bb-4d53-4a7c-b909-4e79c2146edb"
-					(reference "E1")
+					(reference "#PWR071")
 					(unit 1)
 				)
@@
 		(pin "20"
 		)
+		(pin "VBAT-"
+		)
+		(pin "VBAT+"
+		)
 		(instances
 			(project ""
@@
 					(unit 1)
 				)
+			)
+		)
+	)
+	(symbol
+		(lib_id "power:+BATT")
+		(at 274.32 31.75 270)
+		(unit 1)
+		(exclude_from_sim no)
+		(in_bom yes)
+		(on_board yes)
+		(dnp no)
+		(fields_autoplaced yes)
+		(property "Reference" "#PWR070"
+			(at 270.51 31.75 0)
+			(effects
+				(font
+					(size 1.27 1.27)
+				)
+				(hide yes)
+			)
+		)
+		(property "Value" "VBAT+"
+			(at 278.13 31.7499 90)
+			(effects
+				(font
+					(size 1.27 1.27)
+				)
+				(justify left)
+			)
+		)
+		(property "Footprint" ""
+			(at 274.32 31.75 0)
+			(effects
+				(font
+					(size 1.27 1.27)
+				)
+				(hide yes)
+			)
+		)
+		(property "Datasheet" ""
+			(at 274.32 31.75 0)
+			(effects
+				(font
+					(size 1.27 1.27)
+				)
+				(hide yes)
+			)
+		)
+		(property "Description" "Power symbol creates a global label with name \"+BATT\""
+			(at 274.32 31.75 0)
+			(effects
+				(font
+					(size 1.27 1.27)
+				)
+				(hide yes)
+			)
+		)
+		(pin "1"
+		)
+		(instances
+			(project ""
+				(path "/9b6bc1bb-4d53-4a7c-b909-4e79c2146edb"
+					(reference "#PWR070")
+					(unit 1)
+				)
