File: schematic/pcb_left/tk-pie-left.kicad_sch (KiCad schematic)
At the start: 35 parts, among them IC1 PCA9539PW,118, J1 NiceView, J2 Battery Connector, U3 SN74LVC1T45DCK

Commit message: [W.I.P]: Added another battery connector
Also moved around our existing boost circut.
Parts:
- added J3: Battery Connector, Connector_JST:JST_PH_S2B-PH-SM4-TB_1x02-1MP_P2.00mm_Horizontal, symbol Connector:Conn_01x02_Pin
Connections:
- net VBAT+: now also J3.1 (Pin_1)
- net VBAT-: now also J3.2 (Pin_2)
Changed lines of the file:
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@@
 		)
 	)
+	(label "VBAT+"
+		(at 194.31 123.19 0)
+		(effects
+			(font
+				(size 1.27 1.27)
+			)
+			(justify left bottom)
+		)
+	)
 	(label " NV_CS"
 		(at 227.33 44.45 180)
@@
 	)
 	(symbol
+		(lib_id "Connector:Conn_01x02_Pin")
+		(at 189.23 123.19 0)
+		(unit 1)
+		(exclude_from_sim no)
+		(in_bom yes)
+		(on_board yes)
+		(dnp no)
+		(property "Reference" "J3"
+			(at 189.484 119.888 0)
+			(effects
+				(font
+					(size 1.27 1.27)
+				)
+			)
+		)
+		(property "Value" "Battery Connector"
+			(at 188.976 128.778 0)
+			(effects
+				(font
+					(size 1.27 1.27)
+				)
+			)
+		)
+		(property "Footprint" "Connector_JST:JST_PH_S2B-PH-SM4-TB_1x02-1MP_P2.00mm_Horizontal"
+			(at 189.23 123.19 0)
+			(effects
+				(font
+					(size 1.27 1.27)
+				)
+				(hide yes)
+			)
+		)
+		(property "Datasheet" "~"
+			(at 189.23 123.19 0)
+			(effects
+				(font
+					(size 1.27 1.27)
+				)
+				(hide yes)
+			)
+		)
+		(property "Description" "Generic connector, single row, 01x02, script generated"
+			(at 189.23 123.19 0)
+			(effects
+				(font
+					(size 1.27 1.27)
+				)
+				(hide yes)
+			)
+		)
+		(pin "1"
+		)
+		(pin "2"
+		)
+		(instances
+			(project "tk-pie-left"
+				(path "/9b6bc1bb-4d53-4a7c-b909-4e79c2146edb"
+					(reference "J3")
+					(unit 1)
+				)
+			)
+		)
+	)
+	(symbol
 		(lib_id "power:GND")
 		(at 43.18 130.81 180)
@@
 					(unit 1)
 				)
+			)
+		)
+	)
+	(symbol
+		(lib_id "power:GND")
+		(at 194.31 125.73 90)
+		(unit 1)
+		(exclude_from_sim no)
+		(in_bom yes)
+		(on_board yes)
+		(dnp no)
+		(fields_autoplaced yes)
+		(property "Reference" "#PWR072"
+			(at 200.66 125.73 0)
+			(effects
+				(font
+					(size 1.27 1.27)
+				)
+				(hide yes)
+			)
+		)
+		(property "Value" "VBAT-"
+			(at 198.12 125.7299 90)
+			(effects
+				(font
+					(size 1.27 1.27)
+				)
+				(justify right)
+			)
+		)
+		(property "Footprint" ""
+			(at 194.31 125.73 0)
+			(effects
+				(font
+					(size 1.27 1.27)
+				)
+				(hide yes)
+			)
+		)
+		(property "Datasheet" ""
+			(at 194.31 125.73 0)
+			(effects
+				(font
+					(size 1.27 1.27)
+				)
+				(hide yes)
+			)
+		)
+		(property "Description" ""
+			(at 194.31 125.73 0)
+			(effects
+				(font
+					(size 1.27 1.27)
+				)
+				(hide yes)
+			)
+		)
+		(pin "1"
+		)
+		(instances
+			(project "tk-pie-left"
+				(path "/9b6bc1bb-4d53-4a7c-b909-4e79c2146edb"
+					(reference "#PWR072")
+					(unit 1)
+				)

Commit message: Slight updates to battery circuits
Connections:
- net GND: now also J3.2 (Pin_2)
- net VBAT: now also J3.1 (Pin_1)
- net VBAT+: no longer J3.1 (Pin_1)
- net VBAT-: no longer J3.2 (Pin_2)
Changed lines of the file:
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@@
 		)
 	)
-	(label "VBAT+"
+	(label "VBAT"
 		(at 194.31 123.19 0)
 		(effects
@@
 			)
 		)
-		(property "Value" "VBAT-"
+		(property "Value" "GND"
 			(at 198.12 125.7299 90)
 			(effects

Commit message: pcb-left: Fix battery traces
Connections:
- net VBAT is gone; now on net VBAT+: J2.1 (Pin_1), J3.1 (Pin_1)
- net GND: no longer J2.2 (Pin_2), J3.2 (Pin_2)
- net VBAT-: now also J2.2 (Pin_2), J3.2 (Pin_2)
Other:
- note added: "NOTE: Max output is 400mA."
- note removed: "NOTE: Max output is 400mA. is this enough?"
- moved on the sheet: C4, C5, D1, J2, J3, L2, PS1, U3

Commit message: pcb-left: Add name and revision
Other:
- title: (none) -> tk-pie-left
Changed lines of the file:
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@@
 	(generator_version "9.0")
 	(paper "A4")
+	(title_block
+		(title "tk-pie-left")
+		(date "2025-11-09")
+		(rev "2.0")
+	)
 	(rectangle
 		(start 62.23 149.86)
